File: controller/WolfDrive_H7Controller/WolfDrive_H7Controller.sch (KiCad schematic (older format))
At the start: 320 parts, among them CN10 CONN_02X17, CN7 CONN_02X10, CN8 CONN_02X08, CN9 CONN_02X15, CON1 SD_Card, J1 USB_OTG, J10 GND, J11 GND, J12 12VA, J13 Regen, J14 Throttle, J15 PWM1, J16 PWM2, J17 PWM3, J18 ~PWM1, J19 ~PWM2, J2 QSPI_CLK, J20 ~PWM3, J21 OCV, J22 ~F_C, J23 ~F_B, J24 ~F_A, J25 Overtemp, J26 PWM_EN, J27 Conn_01x04_Female, J28 GS3, J29 Conn_01x04, J3 QSPI_NCS, J30 SPI2_SCK, J31 SPI2_NSS, J32 SPI2_MOSI, J33 SPI2_MISO, J34 PS-DIS, J35 3V3, J36 GND, J37 GND, J38 AGND, J39 SP1_MISO, J4 QSPI_IO0, J40 SP1_SCK, J41 SP1_NSS, J42 SP1_MOSI, J43 GS3, J44 GS3, J45 GS3, J46 GS3, J47 GS3, J48 GS3, J49 GS3, J5 QSPI_IO1, J50 GS3, J51 GS3, J52 GS3, J53 GS3, J54 GS3, J55 GS3, J56 GS3, J6 QSPI_IO2, J7 QSPI_IO3, J8 12V, J9 GND, P1 GATE_IO_A, P10 GATE_IO_A, P11 GATE_IO_A, P7 CONN_01X02, P9 GATE_IO_A, U1 LM1117-5.0, U10 74HC266, U11 FT232RL, U12 74LVC1G02, U13 74LVC1G02, U14 74LVC1G02, U15 74LVC1G02, U16 74LVC1G02, U17 74LVC1G02, U18 74LVC1G02, U19 74LVC1G02, U2 LM1117-3.3, U21 74LVC1G02, U3 MCP101-315D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

Commit message: PCB layout progress for issues <5
Parts:
- removed D24: BAT54ADW, TO_SOT_Packages_SMD:SOT-363_SC-70-6_Handsoldering, symbol Diode:BAT54ADW
- added D24, D26: D_Schottky_x2_KCom_AAK, TO_SOT_Packages_SMD:TSOT-23, symbol Device:D_Schottky_x2_KCom_AAK
- added R42: 10k, Resistors_SMD:R_0603_HandSoldering, symbol WolfDrive_H7Controller-rescue:device_R-RESCUE-WolfDrive_H7Controller-WolfDrive_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
- J12: value 12VA -> 5V
Connections:
- net +12VA: no longer J12.1
- net +5V: now also J12.1
- net AGND: now also C69.2
- net DGND: now also R42.1; no longer C69.2
- net Fault_A+: now also D5.1 (K); no longer D5.4 (K)
- net Fault_A-: now also D5.3 (K); no longer D5.5 (K)
- net Fault_B+: now also D19.1 (K); no longer D19.4 (K)
- net Fault_B-: now also D19.3 (K); no longer D19.5 (K)
- net Fault_C+: now also D20.1 (K), I6.1 (R-), R22.2; no longer D20.4 (K), I6.2 (R+), R22.1
- net Fault_C-: now also D20.3 (K), I6.2 (R+), R22.1; no longer D20.5 (K), I6.1 (R-), R22.2
- net GPIO_EXTI14_PF14: now also D24.3 (K), D26.3 (K), R42.2
- net RTD_A+: now also D5.4 (K); no longer D5.3 (K)
- net RTD_A-: now also D5.5 (K); no longer D5.1 (K)
- net RTD_B+: now also D19.4 (K); no longer D19.3 (K)
- net RTD_B-: now also D19.5 (K); no longer D19.1 (K)
- net RTD_C+: now also D20.4 (K); no longer D20.3 (K)
- net RTD_C-: now also D20.5 (K); no longer D20.1 (K)
- net SP1_MISO+: now also D4.3 (K), P1.3 (Pin_3); no longer D4.1 (K), P1.4 (Pin_4)
- net SP1_MISO-: now also D4.4 (K), P1.4 (Pin_4); no longer D4.3 (K), P1.3 (Pin_3)
- net SP1_MOSI+: now also D4.1 (K), P1.5 (Pin_5); no longer D4.5 (K), P1.6 (Pin_6)
- net SP1_MOSI-: now also D4.5 (K), P1.6 (Pin_6); no longer D4.4 (K), P1.5 (Pin_5)
- net SPI1_NSS+: now also P1.9 (Pin_9); no longer P1.8 (Pin_8)
- net SPI1_NSS-: now also P1.10 (Pin_10); no longer P1.7 (Pin_7)
- net SPI1_SCK+: now also P1.7 (Pin_7); no longer P1.10 (Pin_10)
- net SPI1_SCK-: now also P1.8 (Pin_8); no longer P1.9 (Pin_9)
- net at R46.2, U9.1 (Q3): now also D24.2 (A)
- net at R45.2, U9.10 (Q2): now also D26.1 (A)
- net at R39.2, U9.2 (Q0): now also D24.1 (A)
- net at R40.2, U9.9 (Q1): now also D26.2 (A)
Other:
- moved on the sheet: J12
Changed lines of the file:
@@
 	-1   0    0    1
 $EndComp
-Text Label 21650 12250 0    60   ~ 0
+Text Label 21450 12000 0    60   ~ 0
 GPIO_EXTI14_PF14
 Text Label 21675 8050 0    59   ~ 0
@@
 L Connector_Specialized:Test_Point_Flag J12
 U 1 1 5CDBFFB1
-P 5500 3550
-F 0 "J12" H 5558 3670 50  0000 L CNN
-F 1 "12VA" H 5558 3579 50  0000 L CNN
-F 2 "DriveParts:Test_Point" H 5700 3550 50  0001 C CNN
-F 3 "" H 5700 3550 50  0001 C CNN
-	1    5500 3550
+P 6700 1550
+F 0 "J12" H 6758 1670 50  0000 L CNN
+F 1 "5V" H 6758 1579 50  0000 L CNN
+F 2 "DriveParts:Test_Point" H 6900 1550 50  0001 C CNN
+F 3 "" H 6900 1550 50  0001 C CNN
+	1    6700 1550
 	1    0    0    -1
 $EndComp
@@
 Text Label 10750 13575 0    50   ~ 0
 SPI1_NSS-
-Text Label 10200 10400 0    60   ~ 0
-SP1_MOSI+
 Text Label 9700 10400 2    60   ~ 0
+SP1_MOSI+
+Text Label 10200 10400 0    60   ~ 0
 SP1_MOSI-
-Text Label 9700 10600 2    50   ~ 0
+Text Label 10200 10500 0    50   ~ 0
 SPI1_SCK-
-Text Label 10200 10600 0    50   ~ 0
+Text Label 9700 10500 2    50   ~ 0
 SPI1_SCK+
-Text Label 10200 10500 0    50   ~ 0
+Text Label 9700 10600 2    50   ~ 0
 SPI1_NSS+
-Text Label 9700 10500 2    50   ~ 0
+Text Label 10200 10600 0    50   ~ 0
 SPI1_NSS-
-Text Label 9700 10300 2    60   ~ 0
+Text Label 10200 10300 0    60   ~ 0
 SP1_MISO-
 Text Label 11050 8925 0    60   ~ 0
 SP1_MISO+
-Text Label 10200 10300 0    60   ~ 0
+Text Label 9700 10300 2    60   ~ 0
 SP1_MISO+
 $Comp
@@
 Text Label 11275 11625 2    50   ~ 0
 SPI1_NSS-
-Text Label 11300 12100 2    60   ~ 0
+Text Label 11300 12400 2    60   ~ 0
 SP1_MOSI+
-Text Label 11300 12200 2    60   ~ 0
+Text Label 11300 12100 2    60   ~ 0
 SP1_MOSI-
 $Comp
@@
 	0    -1   -1   0
 $EndComp
-Text Label 15650 2675 2    60   ~ 0
+Text Label 15650 2875 2    60   ~ 0
 Fault_A-
-Text Label 15650 2775 2    60   ~ 0
+Text Label 15650 2975 2    60   ~ 0
 Fault_A+
-Text Label 15650 2875 2    60   ~ 0
+Text Label 15650 2775 2    60   ~ 0
 RTD_A+
-Text Label 15650 2975 2    60   ~ 0
+Text Label 15650 2675 2    60   ~ 0
 RTD_A-
 $Comp
@@
 	0    -1   -1   0
 $EndComp
-Text Label 15675 4700 2    60   ~ 0
+Text Label 15675 4900 2    60   ~ 0
 Fault_B-
-Text Label 15675 4800 2    60   ~ 0
+Text Label 15675 5000 2    60   ~ 0
 Fault_B+
-Text Label 15675 4900 2    60   ~ 0
+Text Label 15675 4800 2    60   ~ 0
 RTD_B+
-Text Label 15675 5000 2    60   ~ 0
+Text Label 15675 4700 2    60   ~ 0
 RTD_B-
 $Comp
@@
 	0    -1   -1   0
 $EndComp
-Text Label 15675 6550 2    60   ~ 0
+Text Label 15675 6750 2    60   ~ 0
 Fault_C-
-Text Label 15675 6650 2    60   ~ 0
+Text Label 15675 6850 2    60   ~ 0
 Fault_C+
-Text Label 15675 6750 2    60   ~ 0
+Text Label 15675 6650 2    60   ~ 0
 RTD_C+
-Text Label 15675 6850 2    60   ~ 0
+Text Label 15675 6550 2    60   ~ 0
 RTD_C-
 $Comp
@@
 	0    -1   -1   0
 $EndComp
-Text Label 11300 12300 2    60   ~ 0
+Text Label 11300 12200 2    60   ~ 0
 SP1_MISO-
-Text Label 11300 12400 2    60   ~ 0
+Text Label 11300 12300 2    60   ~ 0
 SP1_MISO+
 Text Notes 14750 1175 0    50   ~ 0
@@
 Text Label 12900 3250 2    60   ~ 0
 Fault_B+
-Text Label 12900 5350 2    60   ~ 0
-Fault_C-
 Text Label 12900 5850 2    60   ~ 0
+Fault_C-
+Text Label 12900 5350 2    60   ~ 0
 Fault_C+
 Text Label 12900 3950 2    60   ~ 0
@@
 $EndComp
 $Comp
-L Diode:BAT54ADW D24
-U 4 1 603F83DE
-P 21650 12450
-F 0 "D24" V 21696 12362 50  0000 R CNN
-F 1 "BAT54ADW" V 21605 12362 50  0000 R CNN
-F 2 "TO_SOT_Packages_SMD:SOT-363_SC-70-6_Handsoldering" H 21650 12275 50  0001 C CNN
-F 3 "http://www.diodes.com/datasheets/ds30152.pdf" H 21650 12550 50  0001 C CNN
-	4    21650 12450
-	0    1    1    0
-$EndComp
-$Comp
 L WolfDrive_H7Controller-rescue:device_R-RESCUE-WolfDrive_H7Controller-WolfDrive_H7Controller-rescue R46
 U 1 1 604008E0
@@
 	-1   0    0    -1
 $EndComp
-$Comp
-L Diode:BAT54ADW D24
-U 2 1 6051D976
-P 21350 12450
-F 0 "D24" V 21396 12362 50  0000 R CNN
-F 1 "BAT54ADW" V 21305 12362 50  0000 R CNN
-F 2 "TO_SOT_Packages_SMD:SOT-363_SC-70-6_Handsoldering" H 21350 12275 50  0001 C CNN
-F 3 "http://www.diodes.com/datasheets/ds30152.pdf" H 21350 12550 50  0001 C CNN
-	2    21350 12450
-	0    1    1    0
-$EndComp
-$Comp
-L Diode:BAT54ADW D24
-U 3 1 6051DC52
-P 21500 12450
-F 0 "D24" V 21546 12362 50  0000 R CNN
-F 1 "BAT54ADW" V 21455 12362 50  0000 R CNN
-F 2 "TO_SOT_Packages_SMD:SOT-363_SC-70-6_Handsoldering" H 21500 12275 50  0001 C CNN
-F 3 "http://www.diodes.com/datasheets/ds30152.pdf" H 21500 12550 50  0001 C CNN
-	3    21500 12450
-	0    1    1    0
-$EndComp
-$Comp
-L Diode:BAT54ADW D24
-U 1 1 6051DF20
-P 21200 12450
-F 0 "D24" V 21246 12362 50  0000 R CNN
-F 1 "BAT54ADW" V 21155 12362 50  0000 R CNN
-F 2 "TO_SOT_Packages_SMD:SOT-363_SC-70-6_Handsoldering" H 21200 12275 50  0001 C CNN
-F 3 "http://www.diodes.com/datasheets/ds30152.pdf" H 21200 12550 50  0001 C CNN
-	1    21200 12450
-	0    1    1    0
-$EndComp
 Wire Wire Line
 	21750 12725 21200 12725
 Wire Wire Line
-	21050 12925 21350 12925
-Wire Wire Line
-	21050 13125 21500 13125
-Wire Wire Line
-	21750 13325 21650 13325
-Wire Wire Line
 	21200 12600 21200 12725
 Connection ~ 21200 12725
 Wire Wire Line
 	21200 12725 21050 12725
-Wire Wire Line
-	21350 12600 21350 12925
-Connection ~ 21350 12925
-Wire Wire Line
-	21350 12925 21750 12925
-Wire Wire Line
-	21500 12600 21500 13125
-Connection ~ 21500 13125
-Wire Wire Line
-	21500 13125 21750 13125
-Wire Wire Line
-	21650 12600 21650 13325
-Connection ~ 21650 13325
-Wire Wire Line
-	21650 13325 21050 13325
-Wire Wire Line
-	21650 12300 21650 12250
-Wire Wire Line
-	21200 12250 21200 12300
-Wire Wire Line
-	21200 12250 21350 12250
-Wire Wire Line
-	21500 12300 21500 12250
-Connection ~ 21500 12250
-Wire Wire Line
-	21500 12250 21650 12250
-Wire Wire Line
-	21350 12300 21350 12250
-Connection ~ 21350 12250
-Wire Wire Line
-	21350 12250 21500 12250
 Connection ~ 6750 2625
 Wire Wire Line
@@
 	5400 3500 5400 3550
 Connection ~ 5400 3550
-$Comp
-L WolfDrive_H7Controller-rescue:WolfDrive_H7Controller-rescue_DGND-RESCUE-WolfDrive_H7Controller-WolfDrive_H7Controller-rescue #PWR0177
-U 1 1 5BC4F7DC
-P 5400 4000
-F 0 "#PWR0177" H 5400 4000 40  0001 C CNN
-F 1 "DGND" H 5400 3930 40  0000 C CNN
-F 2 "" H 5400 4000 60  0000 C CNN
-F 3 "" H 5400 4000 60  0000 C CNN
-	1    5400 4000
-	1    0    0    -1
-$EndComp
 Wire Wire Line
 	5400 3950 5400 4000
@@
 	4600 2625 4600 3550
 Wire Wire Line
-	5850 3550 5500 3550
-Connection ~ 5500 3550
-Wire Wire Line
-	5500 3550 5400 3550
-Wire Wire Line
 	5400 2100 5850 2100
 Wire Wire Line
@@
 	1    0    0    -1
 $EndComp
+$Comp
+L WolfDrive_H7Controller-rescue:device_R-RESCUE-WolfDrive_H7Controller-WolfDrive_H7Controller-rescue R42
+U 1 1 5AE5E213
+P 21450 11750
+F 0 "R42" V 21550 11750 40  0000 C CNN
+F 1 "10k" V 21450 11750 40  0000 C CNN
+F 2 "Resistors_SMD:R_0603_HandSoldering" V 21380 11750 30  0001 C CNN
+F 3 "" H 21450 11750 30  0000 C CNN
+	1    21450 11750
+	1    0    0    -1
+$EndComp
+$Comp
+L Device:D_Schottky_x2_KCom_AAK D24
+U 1 1 5B9D4A33
+P 21200 12300
+F 0 "D24" V 21246 12378 50  0000 L CNN
+F 1 "D_Schottky_x2_KCom_AAK" V 21155 12378 50  0000 L CNN
+F 2 "TO_SOT_Packages_SMD:TSOT-23" H 21200 12300 50  0001 C CNN
+F 3 "~" H 21200 12300 50  0001 C CNN
+	1    21200 12300
+	0    -1   -1   0
+$EndComp
+$Comp
+L Device:D_Schottky_x2_KCom_AAK D26
+U 1 1 5BD3D1F1
+P 21650 12300
+F 0 "D26" V 21604 12379 50  0000 L CNN
+F 1 "D_Schottky_x2_KCom_AAK" V 21695 12379 50  0000 L CNN
+F 2 "TO_SOT_Packages_SMD:TSOT-23" H 21650 12300 50  0001 C CNN
+F 3 "~" H 21650 12300 50  0001 C CNN
+	1    21650 12300
+	0    1    1    0
+$EndComp
+Wire Wire Line
+	21200 12000 21200 11950
+Wire Wire Line
+	21200 11950 21100 11950
+Wire Wire Line
+	21050 13125 21700 13125
+Wire Wire Line
+	21700 13125 21700 11950
+Wire Wire Line
+	21700 11950 21650 11950
+Wire Wire Line
+	21650 11950 21650 12000
+Connection ~ 21700 13125
+Wire Wire Line
+	21700 13125 21750 13125
+Wire Wire Line
+	21400 12300 21450 12300
+Wire Wire Line
+	21450 11900 21450 12300
+Connection ~ 21450 12300
+$Comp
+L WolfDrive_H7Controller-rescue:WolfDrive_H7Controller-rescue_DGND-RESCUE-WolfDrive_H7Controller-WolfDrive_H7Controller-rescue #PWR0183
+U 1 1 5C40EDEA
+P 21450 11600
+F 0 "#PWR0183" H 21450 11600 40  0001 C CNN
+F 1 "DGND" H 21450 11530 40  0000 C CNN
+F 2 "" H 21450 11600 60  0000 C CNN
+F 3 "" H 21450 11600 60  0000 C CNN
+	1    21450 11600
+	1    0    0    1
+$EndComp
+Wire Wire Line
+	21050 12925 21650 12925
+Wire Wire Line
+	21100 11950 21100 13325
+Connection ~ 21100 13325
+Wire Wire Line
+	21100 13325 21050 13325
+Wire Wire Line
+	21100 13325 21750 13325
+Wire Wire Line
+	21650 12600 21650 12925
+Connection ~ 21650 12925
+Wire Wire Line
+	21650 12925 21750 12925
+$Comp
+L WolfDrive_H7Controller-rescue:WolfDrive_H7Controller-rescue_AGND-RESCUE-WolfDrive_H7Controller-WolfDrive_H7Controller-rescue #PWR0177
+U 1 1 5C6763E1
+P 5400 4000
+F 0 "#PWR0177" H 5400 4000 40  0001 C CNN
+F 1 "AGND" H 5400 3900 50  0000 C CNN
+F 2 "" H 5400 4000 60  0000 C CNN
+F 3 "" H 5400 4000 60  0000 C CNN
+	1    5400 4000
+	1    0    0    -1
+$EndComp
+Wire Wire Line
+	5400 3550 5850 3550
+Wire Wire Line
+	6350 1550 6700 1550
 $EndSCHEMATC

Commit message: Major PCB layout revision for v0.2
Parts:
- removed C50: 10n, Capacitors_SMD:C_0603_HandSoldering, symbol WolfDrive_H7Controller-rescue:device_C-RESCUE-WolfDrive_H7Controller-WolfDrive_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
- removed J56: GS3, Connectors:GS3, symbol Jumper:SolderJumper_3_Open
- removed L8: 10uH, Inductors_NEOSID:Neosid_Inductor_SM-NE45_SMD1812, symbol WolfDrive_H7Controller-rescue:WolfDrive_H7Controller-rescue_INDUCTOR_SMALL-RESC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
Connections:
- net +12V: now also D25.1 (A1)
- net +12VA: now also C29.1, C30.1, FI2.3 (VO), L14.1, L15.1
- net DGND: now also D14.1 (K), D15.1 (K), D16.1 (K), D7.1 (K)
- net PWMA_HS+: no longer D22.3 (K)
- net PWMA_HS-: now also D22.3 (K); no longer D22.1 (K)
- net PWMA_LS+: now also D22.5 (K)
- net PWMA_LS-: now also D22.1 (K); no longer D22.5 (K)
- net PWMB_HS+: no longer D23.3 (K)
- net PWMB_HS-: now also D23.3 (K); no longer D23.1 (K)
- net PWMB_LS+: now also D23.5 (K)
- net PWMB_LS-: now also D23.1 (K); no longer D23.5 (K)
- net PWMC_HS+: no longer D21.3 (K)
- net PWMC_HS-: now also D21.3 (K); no longer D21.1 (K)
- net PWMC_LS+: now also D21.5 (K)
- net PWMC_LS-: now also D21.1 (K); no longer D21.5 (K)
- net at F1.2, FL1.2: no longer D25.1 (A1)
Other:
- moved on the sheet: D21, D22, D23, D25, F1
